Commit message: few changes

File: niryo/src/niryo_description/urdf/v2/niryo_one.urdf.xacro (robot description, xacro)
@@ -28,14 +28,20 @@
     <xacro:property name="distance_hand_tool" value="0.0073" />
 	<xacro:property name="PI" value="3.14159265359" />
+    <!-- Joint 1 - Rotation Limit -->
     <xacro:property name="limit_low_shoulder_rotation" value="-3.05433" />
     <xacro:property name="limit_up_shoulder_rotation" value="3.05433" />
+    <!-- Joint 2 - Rotation Limit -->
     <xacro:property name="limit_low_arm_rotation" value="-1.57080" />
     <xacro:property name="limit_up_arm_rotation" value="0.640187" />
+    <!-- Joint 3 - Rotation Limit -->
     <xacro:property name="limit_low_elbow_rotation" value="-1.397485" />
     <xacro:property name="limit_up_elbow_rotation" value="${PI/2}" />
+    <!-- Joint 4 - Rotation Limit -->
     <xacro:property name="limit_low_forearm_rotation" value="-3.05433" />
     <xacro:property name="limit_up_forearm_rotation" value="3.05433" />
+    <!-- Joint 5 - Rotation Limit -->
     <xacro:property name="limit_low_wrist_rotation" value="-1.74533" />
     <xacro:property name="limit_up_wrist_rotation" value="1.91986" />
+    <!-- Joint 6 - Rotation Limit -->
     <xacro:property name="limit_low_hand_rotation" value="-2.57436" />
     <xacro:property name="limit_up_hand_rotation" value="2.57436" />

File: niryo/src/niryo_gazebo/urdf/v2/niryo_one_gazebo.urdf.xacro (robot description, xacro)
@@ -2,5 +2,5 @@
 <robot xmlns:xacro="http://www.ros.org/wiki/xacro" name="niryo_one">
     <!-- Macros -->
-    <xacro:macro name="default_transmission" params="number">
+    <xacro:macro name="default_transmission" params="number reduction">
         <transmission name="transmission_${number}">
             <type>transmission_interface/SimpleTransmission</type>
@@ -10,5 +10,5 @@
             <actuator name="motor_${number}">
                 <hardwareInterface>hardware_interface/PositionJointInterface</hardwareInterface>
-                <mechanicalReduction>1</mechanicalReduction>
+                <mechanicalReduction>${reduction}</mechanicalReduction>
             </actuator>
         </transmission>
@@ -17,10 +17,10 @@
     <xacro:include filename="$(find niryo_description)/urdf/v2/niryo_one.urdf.xacro" />
     <!-- Transmissions-->
-    <xacro:default_transmission number="1"/>
-    <xacro:default_transmission number="2"/>
-    <xacro:default_transmission number="3"/>
-    <xacro:default_transmission number="4"/>
-    <xacro:default_transmission number="5"/>
-    <xacro:default_transmission number="6"/>
+    <xacro:default_transmission number="1" reduction="1"/>
+    <xacro:default_transmission number="2" reduction="1"/>
+    <xacro:default_transmission number="3" reduction="1"/>
+    <xacro:default_transmission number="4" reduction="1"/>
+    <xacro:default_transmission number="5" reduction="1"/>
+    <xacro:default_transmission number="6" reduction="1"/>
     <!-- gazebo ros_control plugin -->
     <gazebo>

Commit message: added radians to step conversion for the first three joints

File: niryo/src/niryo_description/urdf/v2/niryo_one.urdf.xacro (robot description, xacro)
@@ -29,12 +29,12 @@
 	<xacro:property name="PI" value="3.14159265359" />
     <!-- Joint 1 - Rotation Limit -->
-    <xacro:property name="limit_low_shoulder_rotation" value="-3.05433" />
-    <xacro:property name="limit_up_shoulder_rotation" value="3.05433" />
+    <xacro:property name="limit_low_shoulder_rotation" value="-${PI}" />
+    <xacro:property name="limit_up_shoulder_rotation" value="${PI}" />
     <!-- Joint 2 - Rotation Limit -->
-    <xacro:property name="limit_low_arm_rotation" value="-1.57080" />
-    <xacro:property name="limit_up_arm_rotation" value="0.640187" />
+    <xacro:property name="limit_low_arm_rotation" value="-2.355" />
+    <xacro:property name="limit_up_arm_rotation" value="0.628" />
     <!-- Joint 3 - Rotation Limit -->
-    <xacro:property name="limit_low_elbow_rotation" value="-1.397485" />
-    <xacro:property name="limit_up_elbow_rotation" value="${PI/2}" />
+    <xacro:property name="limit_low_elbow_rotation" value="-1.256" />
+    <xacro:property name="limit_up_elbow_rotation" value="1.9625" />
     <!-- Joint 4 - Rotation Limit -->
     <xacro:property name="limit_low_forearm_rotation" value="-3.05433" />

Commit message: added conversion between radians and steps

File: niryo/src/niryo_description/urdf/v2/niryo_one.urdf.xacro (robot description, xacro)
@@ -32,9 +32,9 @@
     <xacro:property name="limit_up_shoulder_rotation" value="${PI}" />
     <!-- Joint 2 - Rotation Limit -->
-    <xacro:property name="limit_low_arm_rotation" value="-2.355" />
-    <xacro:property name="limit_up_arm_rotation" value="0.628" />
+    <xacro:property name="limit_low_arm_rotation" value="-1.6485" />
+    <xacro:property name="limit_up_arm_rotation" value="0.7065" />
     <!-- Joint 3 - Rotation Limit -->
-    <xacro:property name="limit_low_elbow_rotation" value="-1.256" />
-    <xacro:property name="limit_up_elbow_rotation" value="1.9625" />
+    <xacro:property name="limit_low_elbow_rotation" value="-1.3345" />
+    <xacro:property name="limit_up_elbow_rotation" value="2.00175" />
     <!-- Joint 4 - Rotation Limit -->
     <xacro:property name="limit_low_forearm_rotation" value="-3.05433" />
